Commit message: nihao

File: src/my_cartographer/urdf/backpack_2d.urdf (robot description, URDF)
Before this commit: robot drone_model, 3 links, 2 joints
Joints:
- joint imu_joint: origin xyz=0 0 0 rpy=0 0 0 -> xyz=0 0 0.02 rpy=0 0 0
- joint lidar_joint: origin xyz=0 0 0.25 rpy=0 0 0 -> xyz=0 0 0.05 rpy=0 0 0
